File: Sumo_main.sch (EAGLE design)
At the start: 41 parts, among them IC1 TL331, J2 MICRO_USB, T1 0603-PHOTO-TRANS, T2 0603-PHOTO-TRANS, U1 ATMEGA8U2AU, U2 SN65HVD3082, U3 LM339D, X1 MICROMATCH-12, X2 RS485, Y1 16MHz

Commit message: Update main board and schematic
Parts:
- removed D3, D4: IR LED, SparkFun-LED:LED0603
- removed R17, R18: 1K, resistor:R-EU_R0603
- removed R19, R20: 47K, resistor:R-EU_R0603
- removed T1, T2: 0603-PHOTO-TRANS, Phototransistor 0603:0603-PHOTO-TRANS
- added R21, R7: 1K, resistor:R-EU_R0603
- added R4, R5: 47K, resistor:R-EU_R0603
- added U$1, U$2: QRE1113GR, personales:QRE1113GR
Connections:
- removed net N$15: D3.A, R17.1
- removed net N$18: D4.A, R18.1
- new net N$4: R21.1, U$1.A
- new net N$8: R7.1, U$2.A
- net GND: now also J2.P$1, J2.P$2, J2.P$3, J2.P$4, J2.P$5, J2.P$6, U$1.E, U$1.K, U$2.E, U$2.K; no longer D3.C, D4.C, T1.E, T2.E
- net LN1: now also R4.1, U$1.C; no longer R19.1, T1.C
- net LN2: now also R5.1, U$2.C; no longer R20.1, T2.C
- net VCC: now also R21.2, R4.2, R5.2, R7.2; no longer R17.2, R18.2, R19.2, R20.2
